Commit message: fixed 0 value joint-effort limits

File: iiwa_description/urdf/iiwa14.urdf.xacro (robot description, xacro)
@@ -175,5 +175,5 @@
       <child link="${prefix}link_1"/>
       <axis xyz="0 0 1"/>
-      <limit effort="0" lower="-2.9668" upper="2.9668" velocity="1.4834"/>
+      <limit effort="320" lower="-2.9668" upper="2.9668" velocity="1.4834"/>
   </joint>
   <joint name="${prefix}joint_a2" type="revolute">
@@ -182,5 +182,5 @@
       <child link="${prefix}link_2"/>
       <axis xyz="0 1 0"/>
-      <limit effort="0" lower="-2.0942" upper="2.0942" velocity="1.4834"/>
+      <limit effort="320" lower="-2.0942" upper="2.0942" velocity="1.4834"/>
   </joint>
   <joint name="${prefix}joint_a3" type="revolute">
@@ -189,5 +189,5 @@
       <child link="${prefix}link_3"/>
       <axis xyz="0 0 1"/>
-      <limit effort="0" lower="-2.9668" upper="2.9668" velocity="1.7452"/>
+      <limit effort="176" lower="-2.9668" upper="2.9668" velocity="1.7452"/>
   </joint>
   <joint name="${prefix}joint_a4" type="revolute">
@@ -196,5 +196,5 @@
       <child link="${prefix}link_4"/>
       <axis xyz="0 -1 0"/>
-      <limit effort="0" lower="-2.0942" upper="2.0942" velocity="1.3089"/>
+      <limit effort="176" lower="-2.0942" upper="2.0942" velocity="1.3089"/>
   </joint>
   <joint name="${prefix}joint_a5" type="revolute">
@@ -203,5 +203,5 @@
       <child link="${prefix}link_5"/>
       <axis xyz="0 0 1"/>
-      <limit effort="0" lower="-2.9668" upper="2.9668" velocity="2.2688"/>
+      <limit effort="110" lower="-2.9668" upper="2.9668" velocity="2.2688"/>
   </joint>
   <joint name="${prefix}joint_a6" type="revolute">
@@ -210,5 +210,5 @@
       <child link="${prefix}link_6"/>
       <axis xyz="0 1 0"/>
-      <limit effort="0" lower="-2.0942" upper="2.0942" velocity="2.356"/>
+      <limit effort="40" lower="-2.0942" upper="2.0942" velocity="2.356"/>
   </joint>
   <joint name="${prefix}joint_a7" type="revolute">
@@ -217,5 +217,5 @@
       <child link="${prefix}link_7"/>
       <axis xyz="0 0 1"/>
-      <limit effort="0" lower="-3.0541" upper="3.0541" velocity="2.356"/>
+      <limit effort="40" lower="-3.0541" upper="3.0541" velocity="2.356"/>
   </joint>
   <joint name="${prefix}joint_a7-tool0" type="fixed">
