Commit message: added configurable base frame

File: iiwa_description/config/iiwa.config.xacro (robot description, xacro)
@@ -10,4 +10,5 @@
     <xacro:arg name="initial_positions_file" default="initial_positions.yaml" />
     <xacro:arg name="command_interface" default="position" />
+    <xacro:arg name="base_frame_file" default="base_frame.yaml" />
     <!-- Import iiwa urdf file -->
     <xacro:include filename="$(find iiwa_description)/urdf/iiwa14.urdf.xacro" />
@@ -21,6 +22,9 @@
         <static>true</static>
     </gazebo>
+    <xacro:property name="base_frame_file" value="$(arg base_frame_file)"/>
+    <xacro:property name="base_frame" value="${load_yaml(base_frame_file)['base_frame']}"/>
     <xacro:iiwa14 parent="world" prefix="$(arg prefix)">
-        <origin xyz="0 0 0" rpy="0 0 0" />
+        <origin xyz="${base_frame['x']} ${base_frame['y']} ${base_frame['z']}"
+            rpy="${base_frame['roll']} ${base_frame['pitch']} ${base_frame['yaw']}" />
     </xacro:iiwa14>
     <xacro:iiwa_r2c_hardware

Commit message: added namespace to gazebo

File: iiwa_description/config/iiwa.config.xacro (robot description, xacro)
@@ -11,10 +11,14 @@
     <xacro:arg name="command_interface" default="position" />
     <xacro:arg name="base_frame_file" default="base_frame.yaml" />
+    <xacro:arg name="runtime_config_package" default="iiwa_description" />
+    <xacro:arg name="controllers_file" default="iiwa_controllers.yaml" />
+    <xacro:arg name="namespace" default="/" />
+    <xacro:property name="runtime_config_package" value="$(arg runtime_config_package)"/>
     <!-- Import iiwa urdf file -->
-    <xacro:include filename="$(find iiwa_description)/urdf/iiwa14.urdf.xacro" />
+    <xacro:include filename="$(find ${runtime_config_package})/urdf/iiwa14.urdf.xacro" />
     <!-- Import iiwa ros2_control description -->
-    <xacro:include filename="$(find iiwa_description)/ros2_control/iiwa.r2c_hardware.xacro" />
+    <xacro:include filename="$(find ${runtime_config_package})/ros2_control/iiwa.r2c_hardware.xacro" />
     <!-- Import all Gazebo-customization elements -->
-    <xacro:include filename="$(find iiwa_description)/gazebo/iiwa.gazebo"/>
+    <xacro:include filename="$(find ${runtime_config_package})/gazebo/iiwa.gazebo"/>
     <!-- Used for fixing robot -->
     <link name="world"/>
@@ -35,3 +39,8 @@
         use_sim="$(arg use_sim)" use_fake_hardware="$(arg use_fake_hardware)"
         />
+    <!-- <xacro:iiwa_gazebo
+        runtime_config_package="$(arg runtime_config_package)"
+        controllers_file="$(arg controllers_file)"
+        namespace="$(arg namespace)"
+        /> -->
 </robot>

Commit message: added gazebo to main launch (#10)
* added gazebo to main launch

* set up gazebo envar

* fixed broken launch logic

* added configurable base frame

* added namespace handling

* added namespace to gazebo

* fixed gazebo namespace

File: iiwa_description/config/iiwa.config.xacro (robot description, xacro)
@@ -10,10 +10,15 @@
     <xacro:arg name="initial_positions_file" default="initial_positions.yaml" />
     <xacro:arg name="command_interface" default="position" />
+    <xacro:arg name="base_frame_file" default="base_frame.yaml" />
+    <xacro:arg name="runtime_config_package" default="iiwa_description" />
+    <xacro:arg name="controllers_file" default="iiwa_controllers.yaml" />
+    <xacro:arg name="namespace" default="/" />
+    <xacro:property name="runtime_config_package" value="$(arg runtime_config_package)"/>
     <!-- Import iiwa urdf file -->
-    <xacro:include filename="$(find iiwa_description)/urdf/iiwa14.urdf.xacro" />
+    <xacro:include filename="$(find ${runtime_config_package})/urdf/iiwa14.urdf.xacro" />
     <!-- Import iiwa ros2_control description -->
-    <xacro:include filename="$(find iiwa_description)/ros2_control/iiwa.r2c_hardware.xacro" />
+    <xacro:include filename="$(find ${runtime_config_package})/ros2_control/iiwa.r2c_hardware.xacro" />
     <!-- Import all Gazebo-customization elements -->
-    <xacro:include filename="$(find iiwa_description)/gazebo/iiwa.gazebo"/>
+    <xacro:include filename="$(find ${runtime_config_package})/gazebo/iiwa.gazebo.xacro"/>
     <!-- Used for fixing robot -->
     <link name="world"/>
@@ -21,6 +26,9 @@
         <static>true</static>
     </gazebo>
+    <xacro:property name="base_frame_file" value="$(arg base_frame_file)"/>
+    <xacro:property name="base_frame" value="${load_yaml(base_frame_file)['base_frame']}"/>
     <xacro:iiwa14 parent="world" prefix="$(arg prefix)">
-        <origin xyz="0 0 0" rpy="0 0 0" />
+        <origin xyz="${base_frame['x']} ${base_frame['y']} ${base_frame['z']}"
+            rpy="${base_frame['roll']} ${base_frame['pitch']} ${base_frame['yaw']}" />
     </xacro:iiwa14>
     <xacro:iiwa_r2c_hardware
@@ -31,3 +39,9 @@
         use_sim="$(arg use_sim)" use_fake_hardware="$(arg use_fake_hardware)"
         />
+    <xacro:iiwa_gazebo
+        runtime_config_package="$(arg runtime_config_package)"
+        controllers_file="$(arg controllers_file)"
+        namespace="$(arg namespace)"
+        prefix="$(arg prefix)"
+        />
 </robot>

Commit message: renamed iiwa14 to iiwa

File: iiwa_description/config/iiwa.config.xacro (robot description, xacro)
@@ -1,5 +1,5 @@
 <?xml version="1.0"?>
-<!-- Kuka iiwa 14 7DoF manipulator -->
-<robot xmlns:xacro="http://www.ros.org/wiki/xacro" name="iiwa14">
+<!-- Kuka iiwa 7DoF manipulator -->
+<robot xmlns:xacro="http://www.ros.org/wiki/xacro" name="iiwa">
     <!-- Enable setting arguments from the launch file -->
     <xacro:arg name="use_sim" default="false" />
@@ -16,5 +16,5 @@
     <xacro:property name="runtime_config_package" value="$(arg runtime_config_package)"/>
     <!-- Import iiwa urdf file -->
-    <xacro:include filename="$(find ${runtime_config_package})/urdf/iiwa14.urdf.xacro" />
+    <xacro:include filename="$(find ${runtime_config_package})/urdf/iiwa.urdf.xacro" />
     <!-- Import iiwa ros2_control description -->
     <xacro:include filename="$(find ${runtime_config_package})/ros2_control/iiwa.r2c_hardware.xacro" />
@@ -28,8 +28,8 @@
     <xacro:property name="base_frame_file" value="$(arg base_frame_file)"/>
     <xacro:property name="base_frame" value="${load_yaml(base_frame_file)['base_frame']}"/>
-    <xacro:iiwa14 parent="world" prefix="$(arg prefix)">
+    <xacro:iiwa parent="world" prefix="$(arg prefix)">
         <origin xyz="${base_frame['x']} ${base_frame['y']} ${base_frame['z']}"
             rpy="${base_frame['roll']} ${base_frame['pitch']} ${base_frame['yaw']}" />
-    </xacro:iiwa14>
+    </xacro:iiwa>
     <xacro:iiwa_r2c_hardware
         name="iiwaRobot" prefix="$(arg prefix)"

File: iiwa_description/urdf/iiwa.urdf.xacro (robot description, xacro)
@@ -1,5 +1,5 @@
 <?xml version="1.0"?>
 <robot xmlns:xacro="http://www.ros.org/wiki/xacro">
-  <xacro:macro name="iiwa14" params="parent prefix *origin">
+  <xacro:macro name="iiwa" params="parent prefix *origin">
   <material name="gray">
     <color rgba="0.5 0.5 0.5 1.0"/>

Commit message: fixed wrong description package

File: iiwa_description/config/iiwa.config.xacro (robot description, xacro)
@@ -11,14 +11,15 @@
     <xacro:arg name="command_interface" default="position" />
     <xacro:arg name="base_frame_file" default="base_frame.yaml" />
+    <xacro:arg name="description_package" default="iiwa_description" />
     <xacro:arg name="runtime_config_package" default="iiwa_description" />
     <xacro:arg name="controllers_file" default="iiwa_controllers.yaml" />
     <xacro:arg name="namespace" default="/" />
-    <xacro:property name="runtime_config_package" value="$(arg runtime_config_package)"/>
+    <xacro:property name="description_package" value="$(arg description_package)"/>
     <!-- Import iiwa urdf file -->
-    <xacro:include filename="$(find ${runtime_config_package})/urdf/iiwa.urdf.xacro" />
+    <xacro:include filename="$(find ${description_package})/urdf/iiwa.urdf.xacro" />
     <!-- Import iiwa ros2_control description -->
-    <xacro:include filename="$(find ${runtime_config_package})/ros2_control/iiwa.r2c_hardware.xacro" />
+    <xacro:include filename="$(find ${description_package})/ros2_control/iiwa.r2c_hardware.xacro" />
     <!-- Import all Gazebo-customization elements -->
-    <xacro:include filename="$(find ${runtime_config_package})/gazebo/iiwa.gazebo.xacro"/>
+    <xacro:include filename="$(find ${description_package})/gazebo/iiwa.gazebo.xacro"/>
     <!-- Used for fixing robot -->
     <link name="world"/>

Commit message: launch yaml is deprecated

File: iiwa_description/config/iiwa.config.xacro (robot description, xacro)
@@ -28,5 +28,5 @@
     </gazebo>
     <xacro:property name="base_frame_file" value="$(arg base_frame_file)"/>
-    <xacro:property name="base_frame" value="${load_yaml(base_frame_file)['base_frame']}"/>
+    <xacro:property name="base_frame" value="${xacro.load_yaml(base_frame_file)['base_frame']}"/>
     <xacro:iiwa parent="world" prefix="$(arg prefix)">
         <origin xyz="${base_frame['x']} ${base_frame['y']} ${base_frame['z']}"

File: iiwa_description/ros2_control/iiwa.r2c_hardware.xacro (robot description, xacro)
@@ -2,5 +2,5 @@
 <robot xmlns:xacro="http://www.ros.org/wiki/xacro">
     <xacro:macro name="iiwa_r2c_hardware" params="name prefix command_interface robot_ip robot_port initial_positions_file use_sim:=^|false use_fake_hardware:=^|true">
-        <xacro:property name="initial_positions" value="${load_yaml(initial_positions_file)['initial_positions']}"/>
+        <xacro:property name="initial_positions" value="${xacro.load_yaml(initial_positions_file)['initial_positions']}"/>
         <ros2_control name="${name}" type="system">
             <xacro:if value="$(arg use_sim)">

File: iiwa_description/ros2_control/iiwa.r2c_hw_ds.xacro (robot description, xacro)
@@ -2,5 +2,5 @@
 <robot xmlns:xacro="http://www.ros.org/wiki/xacro">
     <xacro:macro name="iiwa_ros2_control" params="name initial_positions_file">
-        <xacro:property name="initial_positions" value="${load_yaml(initial_positions_file)['initial_positions']}"/>
+        <xacro:property name="initial_positions" value="${xacro.load_yaml(initial_positions_file)['initial_positions']}"/>
         <ros2_control name="${name}" type="system">
             <hardware>
