Commit message: add "tip_link" SRDF parameter

File: iiwa_description/srdf/iiwa.srdf.xacro (robot description, xacro)
@@ -6,4 +6,4 @@
   <xacro:property name="description_package" value="$(arg description_package)"/>
   <xacro:include filename="$(find ${description_package})/srdf/iiwa_macro.srdf.xacro"/>
-  <xacro:iiwa_srdf name="$(arg name)" prefix="$(arg prefix)"/>
+  <xacro:iiwa_srdf name="$(arg name)" prefix="$(arg prefix)" tip_link="tool0"/>
 </robot>

File: iiwa_description/srdf/iiwa_macro.srdf.xacro (robot description, xacro)
@@ -1,7 +1,7 @@
 <?xml version="1.0"?>
 <robot xmlns:xacro="http://www.ros.org/wiki/xacro">
-  <xacro:macro name="iiwa_srdf" params="name prefix">
+  <xacro:macro name="iiwa_srdf" params="name prefix tip_link">
      <group name="${prefix}${name}_arm">
-        <chain base_link="${prefix}iiwa_base" tip_link="${prefix}tool0" />
+        <chain base_link="${prefix}iiwa_base" tip_link="${prefix}${tip_link}" />
     </group>
     <group_state name="ready" group="${prefix}${name}_arm">
